File: Shields/Programmer Shield/programmer-shield.brd (EAGLE design)
At the start: 59.7 x 35.6 mm, 6 parts

Commit message: Created gerber files for Core v0.0.6 and re-designed programmer shield
Parts:
- added E$1: (no value), Spark:SPARK_LOGO_PLUS_PLANE
Routing:
- net !RST: track 51.6 -> 38.1 mm, vias 0 -> 3
- net TRST: track 45.5 -> 57.2 mm, vias 0 -> 1
- net TDI: track 37.9 -> 40.2 mm, vias 0 -> 2
- net TCK: track 30.3 -> 31.0 mm
Other:
- board text added: "2013-04-02"
- board text removed: "2013-03-26"
