File: EAGLE/Debug/core-debug.sch (EAGLE design)
At the start: 47 parts, among them Q1 MMDT3904, U1 MIC5219, U3 STM32F10XCXT6, U4 SST25VF040B-50-4I-S2AF, X1 USB-MICROB, Y1 8Mhz

Commit message: Finished Core Debug v0.0.8
Parts:
- added JP3, JP4: (no value), jumper:JP4E
- added JP5, JP6: (no value), jumper:JP2E
- added JP7: (no value), con-harting-ml:ML20
- added JP8, JP9: M12PTH, SparkFun:M12PTH
- added R15, R16, R17, R18: 10K, rcl:R-US_R0603
- added TP1, TP10, TP11, TP2, TP3, TP4, TP5, TP6, TP7, TP8, TP9: TPPAD1-17, testpad:TPPAD1-17
Connections:
- new net BOOT0: JP5.2, U3RESET.BOOT0
- new net BOOT1: JP6.2, U3PORTB_L.PB2
- new net N$11: JP7.19, R17.2
- new net N$12: JP7.11, R15.2
- new net N$14: JP7.17, R16.2
- new net WIFI_RX: JP4.2, U2.WL_RS232_RX
- new net WIFI_TX: JP4.4, U2.WL_RS232_TX
- net !RST: now also JP7.15, JP9.2
- net +3V3: now also JP3.1, JP4.1, JP5.1, JP6.1, JP7.1, JP7.2, JP9.1, R18.2, TP9.TP
- net A0: now also JP8.12
- net A1: now also JP8.11
- net A2: now also JP8.10
- net A3: now also JP8.9
- net A4: now also JP8.8
- net A5: now also JP8.7
- net A6: now also JP8.6
- net A7: now also JP8.5
- net D0: now also JP9.12
- net D1: now also JP9.11
- net D2: now also JP9.10
- net D3: now also JP7.3, JP9.9
- net D4: now also JP7.13, JP9.8, R18.1
- net D5: now also JP7.5, JP9.7
- net D6: now also JP7.9, JP9.6
- net D7: now also JP7.7, JP9.5
- net GND: now also JP3.3, JP4.3, JP5.3, JP6.3, JP7.10, JP7.12, JP7.14, JP7.16, JP7.18, JP7.20, JP7.4, JP7.6, JP7.8, JP8.2, JP9.4, R15.1, R16.1, R17.1, TP10.TP; no longer U3RESET.BOOT0
- net MEM_CS: now also TP7.TP
- net RAW: now also JP8.1
- net RX: now also JP3.2, JP8.4
- net SPI_MISO: now also TP2.TP; no longer U2.SPI_DIN
- net SPI_MOSI: now also TP1.TP, U2.SPI_DIN
- net SPI_SCK: now also TP3.TP
- net TX: now also JP3.4, JP8.3
- net USB_DISC: now also TP6.TP
- net VDDA: now also JP9.3, TP11.TP
- net WIFI_CS: now also TP4.TP
- net WIFI_EN: now also TP8.TP
- net WIFI_INT: now also TP5.TP
Other:
- note added: "Boot Mode Jumpers"
- note added: "CC3000 Serial Interface"
- note added: "Debug Jumpers"
- note added: "JTAG Interface"
- note added: "STM32 Serial Interface"
- moved on the sheet: U3RESET
